File: Molecule_BQ76952 - v2/BMS029B_FETs.kicad_sch (KiCad schematic)
At the start: 135 parts, among them J8 ED555/2DS, J9 OSTTE040161, Q10 MOSFET_N_D3G1S2, Q11 MMBT5401LT1G, Q12 SI7898DP-E3, Q13 MMBT5401LT1G, Q2 SI2325DS-T1-E3, Q3 BSZ900N15NS3 G, Q4 MMBT5401LT1G, Q5 SI2325DS-T1-E3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

Commit message: Final production
Updated sizing and bug fixes
Parts:
- removed J8: ED555/2DS, TERM_BLK_ED555-2DS, symbol Altium Vault - TI:root_0_CMP-0074913-1_Altium Vault - TI
- removed J9: OSTTE040161, FP-OSTTE040161_HDR4-MFG, symbol Altium Vault - TI:root_2_SYM-OSTTE040161_Altium Vault - TI
- added MC25, MC26, MC27, MC28, MC29, MC30: ~, Adom Footprint Library:ADOM_MEDIUM_CONTACT, symbol Adom KiCad Symbols:Adom_Machine_Contact
- Q7: now not fitted
- Q8, Q9: footprint PG-TDSON-8 -> Imported_Parts:BSC033N08NS5SCATMA1
Connections:
- net CPACK+: now also MC29.1, MC30.1
- net PACK+: now also MC25.1, MC26.1
- net PGND: now also MC27.1, MC28.1
