File: Molecule_BQ76952 - v2/BMS029B_Interface.kicad_sch (KiCad schematic)
At the start: 57 parts, among them J24 PBC07SAAN, J25 PBC11SAAN, J26 CONN_USB_5Pos-6Shld, J27 61300211121, J28 PEC05SAAN, J29 22284043, U10 SN74LVC2T45DCTR, U11 CMP-0038965-1, U12 TPD1E10B06DPYT, U13 TPD1E10B06DPYT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

Commit message: Final production
Updated sizing and bug fixes
Parts:
- J24: footprint Sullins_xxC07SAAN -> Kales_Custom_Footprints:ADOM_MEDIUM_HEADER_7
- J25: footprint Sullins_xxC11SAAN -> Kales_Custom_Footprints:ADOM_MEDIUM_HEADER_11
- J27: footprint WURTH_61300211121 -> Kales_Custom_Footprints:ADOM_MEDIUM_HEADER_2
- J29: footprint Molex_0022284043 -> Kales_Custom_Footprints:ADOM_MEDIUM_HEADER_4
Changed lines of the file:
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@@
 			)
 		)
-		(property "Footprint" "Molex_0022284043"
+		(property "Footprint" "Kales_Custom_Footprints:ADOM_MEDIUM_HEADER_4"
 			(at 20.32 215.9 0)
 			(effects
@@
 			)
 		)
-		(property "Footprint" "Sullins_xxC11SAAN"
+		(property "Footprint" "Kales_Custom_Footprints:ADOM_MEDIUM_HEADER_11"
 			(at 27.94 71.12 0)
 			(effects
@@
 			)
 		)
-		(property "Footprint" "Sullins_xxC07SAAN"
+		(property "Footprint" "Kales_Custom_Footprints:ADOM_MEDIUM_HEADER_7"
 			(at 195.58 63.5 0)
 			(effects
@@
 			)
 		)
-		(property "Footprint" "WURTH_61300211121"
+		(property "Footprint" "Kales_Custom_Footprints:ADOM_MEDIUM_HEADER_2"
 			(at 96.52 134.62 0)
 			(effects
