File: Molecule_BQ76952 - v2/BMS029B_PinConfig.kicad_sch (KiCad schematic)
At the start: 31 parts, among them J10 PEC02SAAN, J11 87898-0304, J12 PEC02SAAN, J13 87898-0304, J15 PEC02SAAN, J16 87898-0304, J17 22/05/3041, J18 PEC02SAAN, J19 87898-0304, J20 PEC02SAAN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

Commit message: Final production
Updated sizing and bug fixes
Parts:
- added MC22, MC23, MC24: ~, Adom Footprint Library:ADOM_MEDIUM_CONTACT, symbol Adom KiCad Symbols:Adom_Machine_Contact
- J10, J12, J15, J18, J20, J21: footprint CONN_PEC02SAAN -> Adom Footprint Library:ADOM_JUMPER_4x2
- J11, J13, J16, J19: footprint Molex_87898-0304 -> Adom Footprint Library:ADOM_JUMPER_4x2_3Way_Selector
- J22: footprint Sullins_PxC05SAAN -> Kales_Custom_Footprints:ADOM_MEDIUM_HEADER_5
Connections:
- net PGND: now also MC24.1
- net SCL: now also MC22.1
- net SDA: now also MC23.1
